File: DasarrolloPCB/Proyecto_ELPO_PV.kicad_pcb (KiCad board)
At the start: 2 copper layers, 100 x 100 mm, 32 parts, among them Q1 IRFZ44N, Q2 IRFZ44N, Q3 2N7002, U1 IR2110, U2 IR2110, U3 TL494, U4 ESP32-DEVKITC-32D

Commit message: leyenda ON/OFF arreglada
Parts:
- renumbered ON/OFF to OFF/ON
